Commit message: Add PBVS lock-crop YOLO, frozen-P viz, and 1-DOF ray-scale on the 4s oneshot.
Full-frame top-6 was dropping the locked berry in motion; crop around P0 reprojection recovers a second UV so residual can retarget without cancelling the main traj.

Co-authored-by: Cursor <cursoragent@cursor.com>

File: blueberry_picking_ws/src/picking_description/urdf/suction_eef.urdf.xacro (robot description, xacro)
@@ -1,5 +1,5 @@
 <?xml version="1.0"?>
 <robot xmlns:xacro="http://www.ros.org/wiki/xacro">
-  <!-- Vacuum suction cup: link6 +Z 5cm to eef; cup opens along +Z (real robot / eye-in-hand). -->
+  <!-- Vacuum suction cup: link6 +Z 7cm to eef; cup opens along +Z (real robot / eye-in-hand). -->
   <link name="eef_link">
     <visual>
@@ -20,5 +20,5 @@
     <parent link="link6"/>
     <child link="eef_link"/>
-    <origin xyz="0 0 0.05" rpy="0 0 0"/>
+    <origin xyz="0 0 0.07" rpy="0 0 0"/>
   </joint>
 </robot>

File: blueberry_picking_ws/src/picking_description/urdf/wrist_camera.urdf.xacro (robot description, xacro)
@@ -1,7 +1,6 @@
 <?xml version="1.0"?>
 <robot xmlns:xacro="http://www.ros.org/wiki/xacro">
-  <!-- Wrist Orbbec DaBai on Piper X flange (link6 = 坐标系7 / end-effector fixture).
-       Physical mount: camera on CS7 -Y (~8cm), -Z (~4cm).
-       Optical axis pitched down vs link6 +Z ~23.5deg (roll X); GT fit 20260807_171055. -->
+  <!-- Wrist Orbbec Gemini 305 on Piper X flange (link6).
+       Tape 2026-08-11: (0, -0.07, +0.04). Optical pitch Rx=0 until REFINE tip–berry GT. -->
   <link name="camera_wrist_link">
     <visual>
@@ -20,5 +19,5 @@
     <parent link="link6"/>
     <child link="camera_wrist_link"/>
-    <origin xyz="0 -0.08 -0.04" rpy="-0.410152 0 0"/>
+    <origin xyz="-0.006962964237819408 -0.06433722264599194 0.04" rpy="-0.365480 0.013079 0.094110"/>
   </joint>
   <link name="camera_wrist_color_optical_frame"/>
