Commit message: Refine reach FSM with wrist optical pitch and post-center re-lock.
Apply eye-in-hand Rx≈-23.5° calibration, clear-lock then live cup-aim rebuild after center, and ship refine/contact helper scripts used on the real robot.

Co-authored-by: Cursor <cursoragent@cursor.com>

File: agx_arm_ros/src/agx_arm_description/agx_arm_urdf/piper_x/urdf/piper_x_description.urdf (robot description, URDF)
Before this commit: robot piper_x, 8 links, 7 joints
Joints:
- joint joint6: limit lower=-2.0943951 upper=2.0943951 effort=100 velocity=5 -> lower=0 upper=0 effort=100 velocity=5

File: blueberry_picking_ws/src/picking_description/urdf/wrist_camera.urdf.xacro (robot description, xacro)
@@ -2,6 +2,6 @@
 <robot xmlns:xacro="http://www.ros.org/wiki/xacro">
   <!-- Wrist Orbbec DaBai on Piper X flange (link6 = 坐标系7 / end-effector fixture).
-       Physical mount: camera on CS7 -Y (~8cm); lens Z aligns with CS7 +Z (see install photo).
-       Optical frame = same axes as link6 (no extra rpy); only translation from link6. -->
+       Physical mount: camera on CS7 -Y (~8cm), -Z (~4cm).
+       Optical axis pitched down vs link6 +Z ~23.5deg (roll X); GT fit 20260807_171055. -->
   <link name="camera_wrist_link">
     <visual>
@@ -20,5 +20,5 @@
     <parent link="link6"/>
     <child link="camera_wrist_link"/>
-    <origin xyz="0 -0.08 0" rpy="0 0 0"/>
+    <origin xyz="0 -0.08 -0.04" rpy="-0.410152 0 0"/>
   </joint>
   <link name="camera_wrist_color_optical_frame"/>

Commit message: Add hemisphere occupancy fusion, planner input chain, and fixed-cam calib.
Introduce dual-camera log-odds occupancy in base_link, RViz 3D layers for
OCC/FREE/EGO/ACTIVE fruit, and planner msgs/assembler path for BC cold start.

Co-authored-by: Cursor <cursoragent@cursor.com>

File: agx_arm_ros/src/agx_arm_description/agx_arm_urdf/piper_x/urdf/piper_x_description.urdf (robot description, URDF)
Before this commit: robot piper_x, 8 links, 7 joints
Joints:
- joint joint6: limit lower=0 upper=0 effort=100 velocity=5 -> lower=-2.8797933 upper=2.8797933 effort=100 velocity=5

File: blueberry_picking_ws/src/picking_description/urdf/wrist_camera.urdf.xacro (robot description, xacro)
@@ -19,5 +19,5 @@
     <parent link="link6"/>
     <child link="camera_wrist_link"/>
-    <origin xyz="-0.006962964237819408 -0.06433722264599194 0.04" rpy="-0.365480 0.013079 0.094110"/>
+    <origin xyz="-0.012389519053219772 -0.059366042883212705 0.04" rpy="-0.350288 -0.132947 -0.113574"/>
   </joint>
   <link name="camera_wrist_color_optical_frame"/>
